Commit message: feat:添加tl_hardware并修改moveit相关配置文件实现moveit控制真实机械臂

File: src/tl_moveit2_config/tl_tcb710v_config/config/tl_tcb710v.ros2_control.xacro (robot description, xacro)
@@ -1,10 +1,19 @@
 <?xml version="1.0"?>
 <robot xmlns:xacro="http://www.ros.org/wiki/xacro">
-    <xacro:macro name="tl_tcb710v_ros2_control" params="name initial_positions_file">
-        <xacro:property name="initial_positions" value="${load_yaml(initial_positions_file)['initial_positions']}"/>
+    <xacro:macro name="tl_tcb710v_ros2_control" params="name initial_positions_file use_real_hardware:=false">
+        <xacro:property name="initial_positions" value="${xacro.load_yaml(initial_positions_file)['initial_positions']}"/>
         <ros2_control name="${name}" type="system">
             <hardware>
-                <!-- By default, set up controllers for simulation. This won't work on real hardware -->
-                <plugin>mock_components/GenericSystem</plugin>
+                <xacro:if value="${use_real_hardware}">
+                    <plugin>tl_hardware/TLHardwareInterface</plugin>
+                    <param name="joint_states_topic">/joint_states</param>
+                    <param name="servoj_topic">/tl_driver/set_servoj_pos</param>
+                    <param name="open_servoj_service">/tl_driver/open_servoj</param>
+                    <param name="close_servoj_service">/tl_driver/close_servoj</param>
+                    <param name="state_timeout_sec">1.0</param>
+                </xacro:if>
+                <xacro:unless value="${use_real_hardware}">
+                    <plugin>mock_components/GenericSystem</plugin>
+                </xacro:unless>
             </hardware>
             <joint name="joint1">
